File: ESP32-Adapter/ESP32-Adapter.kicad_pcb (KiCad board)
At the start: 2 copper layers, 0 parts

Commit message: create pcb
Parts:
- added C1: 0.1µ, Capacitor_SMD:C_0402_1005Metric, F.Cu at (114.0, 52.0)
- added C2: 1µ, Capacitor_SMD:C_0402_1005Metric, F.Cu at (94.7, 40.8)
- added D1: D, Diode_SMD:D_0805_2012Metric, F.Cu at (93.8, 37.8)
- added J1: Conn_01x08_Pin, Connector_PinHeader_2.54mm:PinHeader_2x04_P2.54mm_Vertical, F.Cu at (112.9, 99.8)
- added J10: Barrel_Jack, Connector_BarrelJack:BarrelJack_CUI_PJ-063AH_Horizontal, F.Cu at (116.6, 46.0)
- added J12: Conn_01x05, Connector_JST:JST_XH_S5B-XH-A-1_1x05_P2.50mm_Horizontal, F.Cu at (78.0, 119.8)
- added J13: Conn_01x05, Connector_JST:JST_XH_S5B-XH-A-1_1x05_P2.50mm_Horizontal, F.Cu at (96.5, 119.8)
- added J14: Conn_01x04, Connector_JST:JST_XH_S4B-XH-A-1_1x04_P2.50mm_Horizontal, F.Cu at (68.1, 87.5)
- added J2: Conn_01x03, Connector_JST:JST_XH_S3B-XH-A-1_1x03_P2.50mm_Horizontal, F.Cu at (115.4, 89.5)
- added J3: Conn_01x03, Connector_JST:JST_XH_S3B-XH-A-1_1x03_P2.50mm_Horizontal, F.Cu at (115.8, 113.0)
- added R1: 820, Resistor_SMD:R_0402_1005Metric, F.Cu at (94.8, 41.8)
- added R2: 270, Resistor_SMD:R_0402_1005Metric, F.Cu at (94.7, 39.8)
- added U1: ESP32-C5-DevKitC-1, PCM_Espressif:ESP32-C5-DevKitC-1, F.Cu at (70.3, 78.2)
- added U2: LM317_TO-263, Package_TO_SOT_SMD:TO-263-2, F.Cu at (101.8, 40.0)
- added U3: Adafruit CANPAL, Audio_Module:canpal, F.Cu at (71.2, 42.8)
Routing:
- net +5V: track 0.00 -> 140.9 mm, vias 0 -> 1
- net GND: track 0.00 -> 139.2 mm
- net /IDX1: track 0.00 -> 73.8 mm
- net /A1: track 0.00 -> 73.6 mm
- net /B1: track 0.00 -> 73.2 mm
- net /A2: track 0.00 -> 70.6 mm
- net /IDX2: track 0.00 -> 70.3 mm
- net /B2: track 0.00 -> 70.0 mm
- net +3.3V: track 0.00 -> 58.5 mm
- net /SIG2: track 0.00 -> 55.0 mm, vias 0 -> 3
- net /CAN RX: track 0.00 -> 39.6 mm
- net /CAN TX: track 0.00 -> 39.3 mm
- net /SIG1: track 0.00 -> 32.9 mm, vias 0 -> 2
- net Net-(D1-A): track 0.00 -> 24.6 mm
- net Net-(J1-Pin_6): track 0.00 -> 21.4 mm
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