File: ESP32-Adapter/_autosave-ESP32-Adapter.kicad_pcb (KiCad board)
At the start: 2 copper layers, 65.4 x 87.8 mm, 17 parts, among them J10 Barrel_Jack, J12 Conn_01x05, J13 Conn_01x05, J5 Conn_01x03, U1 ESP32-C5-DevKitC-1, U2 LM317DCYR, U3 Adafruit CANPAL, U4 ADAFRUIT INA219 BREAKOUT

Commit message: updates updates
Parts:
- added C3: 0.1µ, Capacitor_SMD:C_0402_1005Metric, F.Cu at (204.6, 30.1)
- added C4: 0.1µ, Capacitor_SMD:C_0402_1005Metric, F.Cu at (204.6, 32.0)
- added U5: ESP32-S3-DevKitC, PCM_Espressif:ESP32-S3-DevKitC, F.Cu at (171.6, 32.5)
